File: ridge_wallet.kicad_pcb (KiCad board)
At the start: 2 copper layers, 86.1 x 53.7 mm, 7 parts

Commit message: Tune the dimensions
Parts:
- moved H2 0.20 mm to (3.30, -50.4)
- moved H4 0.20 mm to (43.0, -50.4)
- moved H6 0.20 mm to (82.5, -50.4)
Routing:
- added copper zone on B.Cu, net (none)
- added copper zone on F.Cu, net (none)
Other:
- board size 86.1 x 53.7 mm -> 86.1 x 53.9 mm
Changed lines of the file:
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@@
   (page A4)
   (layers
-    (0 F.Cu signal)
-    (31 B.Cu signal)
+    (0 F.Cu signal hide)
+    (31 B.Cu signal hide)
     (32 B.Adhes user)
     (33 F.Adhes user)
@@
   )
   (module ridge_wallet:MountingHole_2.5mm (layer F.Cu)
-    (at 82.55 -50.1904)
+    (at 82.55 -50.3904)
     (descr "Mounting Hole 2.5mm, no annular")
     (tags "mounting hole 2.5mm no annular")
@@
   )
   (module ridge_wallet:MountingHole_2.5mm (layer F.Cu)
-    (at 43.05 -50.1904)
+    (at 43.05 -50.3904)
     (descr "Mounting Hole 2.5mm, no annular")
     (tags "mounting hole 2.5mm no annular")
@@
   )
   (module ridge_wallet:MountingHole_2.5mm (layer F.Cu)
-    (at 3.302 -50.1904)
+    (at 3.302 -50.3904)
     (descr "Mounting Hole 2.5mm, no annular")
     (tags "mounting hole 2.5mm no annular")
@@
   (gr_arc (start 59.5 -1.5) (end 59.5 0) (angle -90) (layer Edge.Cuts) (width 0.05))
   (gr_line (start 81 0) (end 83.1 0) (layer Edge.Cuts) (width 0.05))
-  (gr_arc (start 3 -50.7476) (end 3 -53.7476) (angle -90) (layer Edge.Cuts) (width 0.05))
-  (gr_arc (start 83.1 -50.7476) (end 86.1 -50.7476) (angle -90) (layer Edge.Cuts) (width 0.05))
+  (gr_arc (start 3 -50.9476) (end 3 -53.9476) (angle -90) (layer Edge.Cuts) (width 0.05))
+  (gr_arc (start 83.1 -50.9476) (end 86.1 -50.9476) (angle -90) (layer Edge.Cuts) (width 0.05))
   (gr_arc (start 83.1 -3) (end 83.1 0) (angle -90) (layer Edge.Cuts) (width 0.05))
   (gr_arc (start 3 -3) (end 0 -3) (angle -90) (layer Edge.Cuts) (width 0.05))
   (gr_line (start 59.5 0) (end 3 0) (layer Edge.Cuts) (width 0.05))
-  (gr_line (start 86.1 -50.7476) (end 86.1 -3) (layer Edge.Cuts) (width 0.05))
-  (gr_line (start 3 -53.7476) (end 83.1 -53.7476) (layer Edge.Cuts) (width 0.05))
-  (gr_line (start 0 -3) (end 0 -50.7476) (layer Edge.Cuts) (width 0.05))
+  (gr_line (start 86.1 -50.9476) (end 86.1 -3) (layer Edge.Cuts) (width 0.05))
+  (gr_line (start 3 -53.9476) (end 83.1 -53.9476) (layer Edge.Cuts) (width 0.05))
+  (gr_line (start 0 -3) (end 0 -50.9476) (layer Edge.Cuts) (width 0.05))
+  (zone (net 0) (net_name "") (layer F.Cu) (hatch edge 0.508)
+    (connect_pads (clearance 0.508))
+    (min_thickness 0.254)
+    (fill yes (arc_segments 32) (thermal_gap 0.508) (thermal_bridge_width 0.508))
+    (polygon
+      (pts
+        (xy 86.3 0) (xy 0 0) (xy 0 -53.9) (xy 86.3 -53.9)
+      )
+    )
+  )
+  (zone (net 0) (net_name "") (layer B.Cu) (hatch edge 0.508)
+    (connect_pads (clearance 0.508))
+    (min_thickness 0.254)
+    (fill yes (arc_segments 32) (thermal_gap 0.508) (thermal_bridge_width 0.508))
+    (polygon
+      (pts
+        (xy 86.3 0) (xy 0 0) (xy 0 -53.9) (xy 86.3 -53.9)
+      )
+    )
+  )
 )
